File: Layout Eagle/LeiraBoard.sch (EAGLE design)
At the start: 2 parts

Commit message: Leira Board com esquemático terminado e layout feito
Parts:
- added PINOS_METANO, PINOS_TEMPERATURA, PINOS_UMIDADE: (no value), con-lstb:MA03-1
Connections:
- net ANA_METANO: now also PINOS_METANO.2
- net ANA_UMIDADE: now also PINOS_UMIDADE.2
- net GND: now also J1.5, PINOS_METANO.1, PINOS_TEMPERATURA.1, PINOS_UMIDADE.1; no longer J1.9
- net TEMPERATURA: now also PINOS_TEMPERATURA.2
- net VCC: now also PINOS_METANO.3, PINOS_TEMPERATURA.3, PINOS_UMIDADE.3
Other:
- moved on the sheet: J1

Commit message: Atualização LeiraBoard
Parts:
- removed PINOS_UMIDADE: (no value), con-lstb:MA03-1
- added SV1: (no value), con-lstb:MA04-1
Connections:
- net ANA_UMIDADE: now also SV1.1; no longer PINOS_UMIDADE.2
- net GND: now also SV1.3; no longer PINOS_UMIDADE.1
- net VCC: now also SV1.4; no longer PINOS_UMIDADE.3
Changed lines of the file:
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@@
 <part name="GND2" library="SparkFun-PowerSymbols" deviceset="GND" device=""/>
 <part name="PINOS_METANO" library="con-lstb" library_urn="urn:adsk.eagle:library:162" deviceset="MA03-1" device="" package3d_urn="urn:adsk.eagle:package:8339/1"/>
-<part name="PINOS_UMIDADE" library="con-lstb" library_urn="urn:adsk.eagle:library:162" deviceset="MA03-1" device="" package3d_urn="urn:adsk.eagle:package:8339/1"/>
 <part name="SUPPLY3" library="SparkFun-PowerSymbols" deviceset="VCC" device=""/>
 <part name="SUPPLY4" library="SparkFun-PowerSymbols" deviceset="VCC" device=""/>
@@
 <part name="GND5" library="SparkFun-PowerSymbols" deviceset="GND" device=""/>
 <part name="FRAME2" library="frames" library_urn="urn:adsk.eagle:library:229" deviceset="DINA5_L" device=""/>
+<part name="SV1" library="con-lstb" library_urn="urn:adsk.eagle:library:162" deviceset="MA04-1" device="" package3d_urn="urn:adsk.eagle:package:8337/1"/>
 </parts>
 <sheets>
@@
 <instance part="GND2" gate="1" x="162.56" y="96.52"/>
 <instance part="PINOS_METANO" gate="G$1" x="48.26" y="104.14"/>
-<instance part="PINOS_UMIDADE" gate="G$1" x="48.26" y="78.74"/>
 <instance part="SUPPLY3" gate="G$1" x="68.58" y="111.76"/>
 <instance part="SUPPLY4" gate="G$1" x="68.58" y="86.36"/>
 <instance part="GND3" gate="1" x="68.58" y="96.52"/>
-<instance part="GND4" gate="1" x="68.58" y="71.12"/>
+<instance part="GND4" gate="1" x="68.58" y="68.58"/>
 <instance part="PINOS_TEMPERATURA" gate="G$1" x="48.26" y="129.54"/>
 <instance part="SUPPLY5" gate="G$1" x="68.58" y="137.16"/>
 <instance part="GND5" gate="1" x="68.58" y="121.92"/>
 <instance part="FRAME2" gate="G$1" x="22.86" y="35.56"/>
+<instance part="SV1" gate="1" x="48.26" y="78.74"/>
 </instances>
 <busses>
@@
 <pinref part="SUPPLY4" gate="G$1" pin="VCC"/>
 <wire x1="68.58" y1="81.28" x2="68.58" y2="86.36" width="0.1524" layer="91"/>
-<pinref part="PINOS_UMIDADE" gate="G$1" pin="3"/>
 <wire x1="55.88" y1="81.28" x2="68.58" y2="81.28" width="0.1524" layer="91"/>
 <label x="55.88" y="81.28" size="1.778" layer="95"/>
+<pinref part="SV1" gate="1" pin="4"/>
 </segment>
 <segment>
@@
 </segment>
 <segment>
-<pinref part="PINOS_UMIDADE" gate="G$1" pin="2"/>
-<wire x1="55.88" y1="78.74" x2="66.04" y2="78.74" width="0.1524" layer="91"/>
-<label x="55.88" y="78.74" size="1.778" layer="95"/>
+<wire x1="55.88" y1="73.66" x2="66.04" y2="73.66" width="0.1524" layer="91"/>
+<label x="55.88" y="73.66" size="1.778" layer="95"/>
+<pinref part="SV1" gate="1" pin="1"/>
 </segment>
 </net>
@@
 </segment>
 <segment>
-<pinref part="PINOS_UMIDADE" gate="G$1" pin="1"/>
-<wire x1="68.58" y1="76.2" x2="55.88" y2="76.2" width="0.1524" layer="91"/>
-<label x="55.88" y="76.2" size="1.778" layer="95"/>
+<wire x1="68.58" y1="78.74" x2="55.88" y2="78.74" width="0.1524" layer="91"/>
+<label x="55.88" y="78.74" size="1.778" layer="95"/>
 <pinref part="GND4" gate="1" pin="GND"/>
-<wire x1="68.58" y1="76.2" x2="68.58" y2="73.66" width="0.1524" layer="91"/>
+<wire x1="68.58" y1="78.74" x2="68.58" y2="71.12" width="0.1524" layer="91"/>
+<pinref part="SV1" gate="1" pin="3"/>
 </segment>
 <segment>
